File: MAX31850K_Breakout/MAX31850K_breakout.brd (EAGLE design)
At the start: 20 x 20 mm, 6 parts, among them U1 3.3V

Commit message: Almost have all components created in LoganSmith-Eagle-Library.
Parts:
- added AD0, AD1, AD2, AD3: (no value), LoganSmith-Connectors:SJ_3
- added J1: M08SQ1, LoganSmith-Connectors:1X08_SQ1
- added LOGO1: OSHW-LOGOM, SparkFun-Aesthetics:OSHW-LOGO-M
- added U$1, U$2: MNTHOLE-2.0, LoganSmith-Electromechanical:MOUNTINGHOLE_2.0_PLATED
- added U2: MAX31850K, LoganSmith-Digital_IC:10-TDFN-EP
- moved C3 3.81 mm to (14.0, 17.8)
- moved U1 3.81 mm to (10.2, 17.8)
- moved C2 2.54 mm to (6.35, 16.5)
Connections:
- removed net N$1: C1.P$1
- removed net N$2: C1.P$2
- new net AD0: AD0.2, J1.4, U2.6
- new net AD1: AD1.2, J1.5, U2.7
- new net AD2: AD2.2, J1.6, U2.8
- new net AD3: AD3.2, J1.7, U2.9
- new net DATA: AD0.1, AD1.1, AD2.1, AD3.1, J1.8, U2.5
- new net TM_FILT: C1.P$2, FB2.P$2, U2.2
- new net TP_FILT: C1.P$1, FB1.P$2, U2.3
- new net VIN: C2.P$3, J1.2, U1.1, U1.3
- net +3V3: now also J1.3, U2.4; no longer C2.P$3, U1.1, U1.3
- net GND: now also AD0.3, AD1.3, AD2.3, AD3.3, J1.1, U$1.P$1, U$2.P$1, U2.1, U2.PAD
Other:
- board text added: "0"
- board text added: "1"
- board text added: "MAX31851K"
- board text added: "Red -"
- board text added: "Yellow +"
- board text added: "v1.0"
