File: MAX31850K_Breakout/MAX31850K_breakout.sch (EAGLE design)
At the start: 6 parts, among them U1 3.3V

Commit message: Almost have all components created in LoganSmith-Eagle-Library.
Parts:
- added AD0, AD1, AD2, AD3: (no value), LoganSmith-Connectors:SJ_2WAYS
- added J1: M08SQ1, LoganSmith-Connectors:M08SQ1
- added LOGO1: OSHW-LOGOM, SparkFun-Aesthetics:OSHW-LOGOM
- added U$1, U$2: MNTHOLE-2.0, LoganSmith-Electromechanical:MNTHOLE-2.0
- added U2: MAX31850K, LoganSmith-Digital_IC:MAX31850K
Connections:
- removed net N$1: C1.1
- removed net N$2: C1.2
- new net AD0: AD0.2, J1.4, U2.AD0
- new net AD1: AD1.2, J1.5, U2.AD1
- new net AD2: AD2.2, J1.6, U2.AD2
- new net AD3: AD3.2, J1.7, U2.AD3
- new net DATA: AD0.1, AD1.1, AD2.1, AD3.1, J1.8, U2.DQ
- new net TM_FILT: C1.2, FB2.2, U2.T-
- new net TP_FILT: C1.1, FB1.2, U2.T+
- new net VIN: C2.1, J1.2, U1.EN, U1.VIN
- net +3V3: now also J1.3, U2.VDD; no longer C2.1, U1.EN, U1.VIN
- net GND: now also AD0.3, AD1.3, AD2.3, AD3.3, J1.1, U$1.P$1, U$2.P$1, U2.GND, U2.PAD
